File: KiCad-Project/ESP32/ESP32.sch (KiCad schematic (older format))
At the start: 16 parts, among them J3 UART, SW1 RESET, U3 AMS1117-3.3, U4 ESP32-WROOM-32

Commit message: Move on board test LED to a better pin. and swap TX/RX UART pins
Connections:
- net IO19 is gone; now on an unnamed net: U4.31 (IO19)
- net UART_RX: now also J3.4 (Pin_4); no longer J3.5 (Pin_5)
- net UART_TX: now also J3.5 (Pin_5); no longer J3.4 (Pin_4)
- net at R10.1: no longer U4.16 (IO13)
- no-connect marks 18 -> 19
Other:
- moved on the sheet: LED2, R10
Changed lines of the file:
@@
 Text Label 9350 1750 0    50   ~ 0
 CTS
+Text Label 9350 2050 0    50   ~ 0
+UART_TX
 Text Label 9350 1950 0    50   ~ 0
-UART_TX
-Text Label 9350 2050 0    50   ~ 0
 UART_RX
 Text Label 9350 2150 0    50   ~ 0
@@
 L Device:LED LED2
 U 1 1 618A3283
-P 9500 2550
-F 0 "LED2" H 9625 2425 50  0000 R CNN
-F 1 "IO13_LED" H 9700 2700 50  0000 R CNN
-F 2 "LED_SMD:LED_0805_2012Metric" H 9500 2550 50  0001 C CNN
-F 3 "~" H 9500 2550 50  0001 C CNN
-F 4 "C84256" H 9500 2550 50  0001 C CNN "JLCPCB_PNUM"
-F 5 "NCD0805R1" H 9500 2550 50  0001 C CNN "MFG_PNUM"
-F 6 "LED_0805" H 9500 2550 50  0001 C CNN "PACKAGE"
-F 7 "JLCPCB" H 9500 2550 50  0001 C CNN "SUPPLIER"
-	1    9500 2550
+P 9650 3150
+F 0 "LED2" H 9775 3025 50  0000 R CNN
+F 1 "IO13_LED" H 9850 3300 50  0000 R CNN
+F 2 "LED_SMD:LED_0805_2012Metric" H 9650 3150 50  0001 C CNN
+F 3 "~" H 9650 3150 50  0001 C CNN
+F 4 "C84256" H 9650 3150 50  0001 C CNN "JLCPCB_PNUM"
+F 5 "NCD0805R1" H 9650 3150 50  0001 C CNN "MFG_PNUM"
+F 6 "LED_0805" H 9650 3150 50  0001 C CNN "PACKAGE"
+F 7 "JLCPCB" H 9650 3150 50  0001 C CNN "SUPPLIER"
+	1    9650 3150
 	-1   0    0    1
 $EndComp
@@
 L Device:R_Small R10
 U 1 1 618A7BBE
-P 9150 2550
-F 0 "R10" V 9050 2500 50  0000 L CNN
-F 1 "200" V 9250 2500 50  0000 L CNN
-F 2 "Resistor_SMD:R_0805_2012Metric" H 9150 2550 50  0001 C CNN
-F 3 "~" H 9150 2550 50  0001 C CNN
-F 4 "C17540" H 9150 2550 50  0001 C CNN "JLCPCB_PNUM"
-F 5 "0805W8F2000T5E" H 9150 2550 50  0001 C CNN "MFG_PNUM"
-F 6 "0805" H 9150 2550 50  0001 C CNN "PACKAGE"
-F 7 "JLCPCB" H 9150 2550 50  0001 C CNN "SUPPLIER"
-	1    9150 2550
+P 9300 3150
+F 0 "R10" V 9200 3100 50  0000 L CNN
+F 1 "200" V 9400 3100 50  0000 L CNN
+F 2 "Resistor_SMD:R_0805_2012Metric" H 9300 3150 50  0001 C CNN
+F 3 "~" H 9300 3150 50  0001 C CNN
+F 4 "C17540" H 9300 3150 50  0001 C CNN "JLCPCB_PNUM"
+F 5 "0805W8F2000T5E" H 9300 3150 50  0001 C CNN "MFG_PNUM"
+F 6 "0805" H 9300 3150 50  0001 C CNN "PACKAGE"
+F 7 "JLCPCB" H 9300 3150 50  0001 C CNN "SUPPLIER"
+	1    9300 3150
 	0    -1   1    0
 $EndComp
 Wire Wire Line
-	9350 2550 9250 2550
-Wire Wire Line
-	9800 2550 9650 2550
+	9500 3150 9400 3150
+Wire Wire Line
+	9950 3150 9800 3150
 $Comp
 L power:GND #PWR017
@@
 Text Label 8700 1850 2    50   ~ 0
 ~FLASH
-Wire Wire Line
-	8350 1950 9700 1950
 Wire Notes Line
 	850  2950 850  4700
@@
 Text Label 9350 1850 0    50   ~ 0
 UART_VCC
-Wire Wire Line
-	8775 2050 8775 2150
-Wire Wire Line
-	8775 2150 8350 2150
 Wire Wire Line
 	7750 4450 7750 4600
@@
 Wire Wire Line
 	3800 1350 4300 1350
-Wire Wire Line
-	8775 2050 9700 2050
 Wire Wire Line
 	8350 3350 8525 3350
@@
 SDA
 Wire Wire Line
-	8350 3150 8700 3150
-Wire Wire Line
 	8350 3450 8700 3450
-Text Label 8700 3150 0    50   ~ 0
-IO19
 Text Label 8700 3450 0    50   ~ 0
 IO23
@@
 	8350 2850 8875 2850
 NoConn ~ 8350 2250
-Wire Wire Line
-	8350 2550 9050 2550
 Wire Wire Line
 	3650 3950 4700 3950
@@
 	8650 1500 8825 1500
 $Comp
-L power:GND #PWR?
+L power:GND #PWR0119
 U 1 1 61B80328
-P 9800 2550
-F 0 "#PWR?" H 9800 2300 50  0001 C CNN
-F 1 "GND" V 9805 2422 50  0000 R CNN
-F 2 "" H 9800 2550 50  0001 C CNN
-F 3 "" H 9800 2550 50  0001 C CNN
-	1    9800 2550
+P 9950 3150
+F 0 "#PWR0119" H 9950 2900 50  0001 C CNN
+F 1 "GND" V 9955 3022 50  0000 R CNN
+F 2 "" H 9950 3150 50  0001 C CNN
+F 3 "" H 9950 3150 50  0001 C CNN
+	1    9950 3150
 	0    -1   -1   0
 $EndComp
 $Comp
-L power:+3.3V #PWR?
+L power:+3.3V #PWR0120
 U 1 1 61A96D0C
 P 8650 1500
-F 0 "#PWR?" H 8650 1350 50  0001 C CNN
+F 0 "#PWR0120" H 8650 1350 50  0001 C CNN
 F 1 "+3.3V" H 8665 1673 50  0000 C CNN
 F 2 "" H 8650 1500 50  0001 C CNN
@@
 	0    -1   -1   0
 $EndComp
+Wire Wire Line
+	8350 3150 9200 3150
+NoConn ~ 8350 2550
+Wire Wire Line
+	8350 1950 8550 1950
+Wire Wire Line
+	8550 1950 8550 2050
+Wire Wire Line
+	8550 2050 9700 2050
+Wire Wire Line
+	8350 2150 8900 2150
+Wire Wire Line
+	8900 2150 8900 1950
+Wire Wire Line
+	8900 1950 9700 1950
 $EndSCHEMATC

Commit message: update pin labels
Connections:
- net +3V3: now also LED2.2 (A)
- net GND: no longer LED2.1 (K)
- net at R10.2: now also LED2.1 (K); no longer LED2.2 (A)
Other:
- moved on the sheet: LED2
Changed lines of the file:
@@
 F 7 "JLCPCB" H 9650 3150 50  0001 C CNN "SUPPLIER"
 	1    9650 3150
-	-1   0    0    1
+	1    0    0    1
 $EndComp
 $Comp
@@
 	8650 1500 8825 1500
 $Comp
-L power:GND #PWR0119
-U 1 1 61B80328
-P 9950 3150
-F 0 "#PWR0119" H 9950 2900 50  0001 C CNN
-F 1 "GND" V 9955 3022 50  0000 R CNN
-F 2 "" H 9950 3150 50  0001 C CNN
-F 3 "" H 9950 3150 50  0001 C CNN
-	1    9950 3150
-	0    -1   -1   0
-$EndComp
-$Comp
 L power:+3.3V #PWR0120
 U 1 1 61A96D0C
@@
 Wire Wire Line
 	8900 1950 9700 1950
+$Comp
+L power:+3.3V #PWR0119
+U 1 1 61B19B18
+P 9950 3150
+F 0 "#PWR0119" H 9950 3000 50  0001 C CNN
+F 1 "+3.3V" H 9965 3323 50  0000 C CNN
+F 2 "" H 9950 3150 50  0001 C CNN
+F 3 "" H 9950 3150 50  0001 C CNN
+	1    9950 3150
+	0    1    1    0
+$EndComp
 $EndSCHEMATC
