File: KiCad-Project/ESP32/ESP32.sch (KiCad schematic (older format))
At the start: 16 parts, among them J3 UART, SW1 RESET, U3 AMS1117-3.3, U4 ESP32-WROOM-32

Commit message: Reset annotations
Parts:
- renumbered C9 to C10, C10 to C8, C8 to C9, JP2 to JP10, JP1 to JP9, R8 to R6, R9 to R7, R10 to R8, U3 to U11, U4 to U12
Changed lines of the file:
@@
 $EndDescr
 $Comp
-L Regulator_Linear:AMS1117-3.3 U3
+L Regulator_Linear:AMS1117-3.3 U11
 U 1 1 6186F41D
 P 3350 1350
-F 0 "U3" H 3350 1592 50  0000 C CNN
+F 0 "U11" H 3350 1592 50  0000 C CNN
 F 1 "AMS1117-3.3" H 3350 1501 50  0000 C CNN
 F 2 "Package_TO_SOT_SMD:SOT-223-3_TabPin2" H 3350 1550 50  0001 C CNN
@@
 Power Supply
 $Comp
-L power:+5V #PWR014
+L power:+5V #PWR040
 U 1 1 618736F0
 P 1650 1250
-F 0 "#PWR014" H 1650 1100 50  0001 C CNN
+F 0 "#PWR040" H 1650 1100 50  0001 C CNN
 F 1 "+5V" H 1665 1423 50  0000 C CNN
 F 2 "" H 1650 1250 50  0001 C CNN
@@
 $EndComp
 $Comp
-L power:GND #PWR013
+L power:GND #PWR039
 U 1 1 618740AA
 P 1550 2450
-F 0 "#PWR013" H 1550 2200 50  0001 C CNN
+F 0 "#PWR039" H 1550 2200 50  0001 C CNN
 F 1 "GND" H 1555 2277 50  0000 C CNN
 F 2 "" H 1550 2450 50  0001 C CNN
@@
 	1550 2300 1550 2450
 $Comp
-L Device:R_Small R8
+L Device:R_Small R6
 U 1 1 618765CE
 P 1550 1750
-F 0 "R8" H 1609 1796 50  0000 L CNN
+F 0 "R6" H 1609 1796 50  0000 L CNN
 F 1 "2.2K" H 1609 1705 50  0000 L CNN
 F 2 "Resistor_SMD:R_0805_2012Metric" H 1550 1750 50  0001 C CNN
@@
 Connection ~ 2250 1350
 $Comp
-L power:GND #PWR015
+L power:GND #PWR041
 U 1 1 6187C1EC
 P 2250 2450
-F 0 "#PWR015" H 2250 2200 50  0001 C CNN
+F 0 "#PWR041" H 2250 2200 50  0001 C CNN
 F 1 "GND" H 2255 2277 50  0000 C CNN
 F 2 "" H 2250 2450 50  0001 C CNN
@@
 	2250 1900 2250 2250
 $Comp
-L power:GND #PWR018
+L power:GND #PWR044
 U 1 1 6187D2F3
 P 3350 2450
-F 0 "#PWR018" H 3350 2200 50  0001 C CNN
+F 0 "#PWR044" H 3350 2200 50  0001 C CNN
 F 1 "GND" H 3355 2277 50  0000 C CNN
 F 2 "" H 3350 2450 50  0001 C CNN
@@
 $EndComp
 $Comp
-L power:+3.3V #PWR019
+L power:+3.3V #PWR045
 U 1 1 6187E501
 P 3800 1250
-F 0 "#PWR019" H 3800 1100 50  0001 C CNN
+F 0 "#PWR045" H 3800 1100 50  0001 C CNN
 F 1 "+3.3V" H 3815 1423 50  0000 C CNN
 F 2 "" H 3800 1250 50  0001 C CNN
@@
 $EndComp
 $Comp
-L Device:C C8
+L Device:C C9
 U 1 1 6187F6DC
 P 3800 1750
-F 0 "C8" H 3915 1796 50  0000 L CNN
+F 0 "C9" H 3915 1796 50  0000 L CNN
 F 1 "0.1uF" H 3915 1705 50  0000 L CNN
 F 2 "Capacitor_SMD:C_0805_2012Metric" H 3838 1600 50  0001 C CNN
@@
 Connection ~ 3800 1350
 $Comp
-L power:GND #PWR020
+L power:GND #PWR046
 U 1 1 61880862
 P 3800 2450
-F 0 "#PWR020" H 3800 2200 50  0001 C CNN
+F 0 "#PWR046" H 3800 2200 50  0001 C CNN
 F 1 "GND" H 3805 2277 50  0000 C CNN
 F 2 "" H 3800 2450 50  0001 C CNN
@@
 	850  650  850  2850
 $Comp
-L power:GND #PWR028
+L power:GND #PWR051
 U 1 1 61889385
 P 9350 1650
-F 0 "#PWR028" H 9350 1400 50  0001 C CNN
+F 0 "#PWR051" H 9350 1400 50  0001 C CNN
 F 1 "GND" V 9355 1522 50  0000 R CNN
 F 2 "" H 9350 1650 50  0001 C CNN
@@
 UART_RTS
 $Comp
-L power:GND #PWR025
+L power:GND #PWR049
 U 1 1 6188BB8F
 P 7750 4600
-F 0 "#PWR025" H 7750 4350 50  0001 C CNN
+F 0 "#PWR049" H 7750 4350 50  0001 C CNN
 F 1 "GND" H 7755 4427 50  0000 C CNN
 F 2 "" H 7750 4600 50  0001 C CNN
@@
 $EndComp
 $Comp
-L power:+3.3V #PWR024
+L power:+3.3V #PWR048
 U 1 1 6188C5C7
 P 7750 1450
-F 0 "#PWR024" H 7750 1300 50  0001 C CNN
+F 0 "#PWR048" H 7750 1300 50  0001 C CNN
 F 1 "+3.3V" H 7765 1623 50  0000 C CNN
 F 2 "" H 7750 1450 50  0001 C CNN
@@
 	2300 3850 2575 3850
 $Comp
-L power:GND #PWR012
+L power:GND #PWR038
 U 1 1 6189DEED
 P 1200 4450
-F 0 "#PWR012" H 1200 4200 50  0001 C CNN
+F 0 "#PWR038" H 1200 4200 50  0001 C CNN
 F 1 "GND" H 1205 4277 50  0000 C CNN
 F 2 "" H 1200 4450 50  0001 C CNN
@@
 	1200 4250 1200 4450
 $Comp
-L Device:R_Small R9
+L Device:R_Small R7
 U 1 1 6189F74B
 P 2300 3550
-F 0 "R9" H 2359 3596 50  0000 L CNN
+F 0 "R7" H 2359 3596 50  0000 L CNN
 F 1 "10K" H 2359 3505 50  0000 L CNN
 F 2 "Resistor_SMD:R_0805_2012Metric" H 2300 3550 50  0001 C CNN
@@
 	2300 3850 2300 3650
 $Comp
-L power:+3.3V #PWR016
+L power:+3.3V #PWR042
 U 1 1 618A1713
 P 2300 3300
-F 0 "#PWR016" H 2300 3150 50  0001 C CNN
+F 0 "#PWR042" H 2300 3150 50  0001 C CNN
 F 1 "+3.3V" H 2315 3473 50  0000 C CNN
 F 2 "" H 2300 3300 50  0001 C CNN
@@
 NoConn ~ 9350 2150
 $Comp
-L Device:C C9
+L Device:C C10
 U 1 1 6189C75C
 P 4300 1750
-F 0 "C9" H 4415 1796 50  0000 L CNN
+F 0 "C10" H 4415 1796 50  0000 L CNN
 F 1 "10uf" H 4415 1705 50  0000 L CNN
 F 2 "Capacitor_SMD:C_0805_2012Metric" H 4338 1600 50  0001 C CNN
@@
 $EndComp
 $Comp
-L power:GND #PWR021
+L power:GND #PWR047
 U 1 1 6189CEF4
 P 4300 2450
-F 0 "#PWR021" H 4300 2200 50  0001 C CNN
+F 0 "#PWR047" H 4300 2200 50  0001 C CNN
 F 1 "GND" H 4305 2277 50  0000 C CNN
 F 2 "" H 4300 2450 50  0001 C CNN
@@
 $EndComp
 $Comp
-L Device:R_Small R10
+L Device:R_Small R8
 U 1 1 618A7BBE
 P 9300 3150
-F 0 "R10" V 9200 3100 50  0000 L CNN
+F 0 "R8" V 9200 3100 50  0000 L CNN
 F 1 "200" V 9400 3100 50  0000 L CNN
 F 2 "Resistor_SMD:R_0805_2012Metric" H 9300 3150 50  0001 C CNN
@@
 	9950 3150 9800 3150
 $Comp
-L power:GND #PWR017
+L power:GND #PWR043
 U 1 1 618BCAB2
 P 3100 4100
-F 0 "#PWR017" H 3100 3850 50  0001 C CNN
+F 0 "#PWR043" H 3100 3850 50  0001 C CNN
 F 1 "GND" H 3105 3927 50  0000 C CNN
 F 2 "" H 3100 4100 50  0001 C CNN
@@
 	7150 1850 6800 1850
 $Comp
-L RF_Module:ESP32-WROOM-32 U4
+L RF_Module:ESP32-WROOM-32 U12
 U 1 1 618CD539
 P 7750 3050
-F 0 "U4" H 7275 4400 50  0000 C CNN
+F 0 "U12" H 7275 4400 50  0000 C CNN
 F 1 "ESP32-WROOM-32" H 8150 4425 50  0000 C CNN
 F 2 "RF_Module:ESP32-WROOM-32" H 7750 1550 50  0001 C CNN
@@
 	3350 1650 3350 2450
 $Comp
-L power:PWR_FLAG #FLG0103
+L power:PWR_FLAG #FLG03
 U 1 1 6193BC34
 P 2575 3850
-F 0 "#FLG0103" H 2575 3925 50  0001 C CNN
+F 0 "#FLG03" H 2575 3925 50  0001 C CNN
 F 1 "PWR_FLAG" H 2575 4023 50  0000 C CNN
 F 2 "" H 2575 3850 50  0001 C CNN
@@
 	3100 3950 3450 3950
 $Comp
-L Device:Jumper_NO_Small JP1
+L Device:Jumper_NO_Small JP9
 U 1 1 6189F27D
 P 3550 3950
-F 0 "JP1" H 3550 4135 50  0000 C CNN
+F 0 "JP9" H 3550 4135 50  0000 C CNN
 F 1 "FLASH" H 3550 4044 50  0000 C CNN
 F 2 "Connector_PinHeader_2.54mm:PinHeader_1x02_P2.54mm_Vertical" H 3550 3950 50  0001 C CNN
@@
 $EndComp
 $Comp
-L Device:C C10
+L Device:C C8
 U 1 1 61B24BD4
 P 2750 1750
-F 0 "C10" H 2865 1796 50  0000 L CNN
+F 0 "C8" H 2865 1796 50  0000 L CNN
 F 1 "22uF" H 2865 1705 50  0000 L CNN
 F 2 "Capacitor_SMD:C_0805_2012Metric" H 2788 1600 50  0001 C CNN
@@
 	2250 2250 2250 2450
 $Comp
-L Device:Jumper_NO_Small JP2
+L Device:Jumper_NO_Small JP10
 U 1 1 61B4F51D
 P 8925 1500
-F 0 "JP2" H 8925 1685 50  0000 C CNN
+F 0 "JP10" H 8925 1685 50  0000 C CNN
 F 1 "UART_VCC" H 8925 1594 50  0000 C CNN
 F 2 "Connector_PinHeader_2.54mm:PinHeader_1x02_P2.54mm_Vertical" H 8925 1500 50  0001 C CNN
@@
 	8650 1500 8825 1500
 $Comp
-L power:+3.3V #PWR0120
+L power:+3.3V #PWR050
 U 1 1 61A96D0C
 P 8650 1500
-F 0 "#PWR0120" H 8650 1350 50  0001 C CNN
+F 0 "#PWR050" H 8650 1350 50  0001 C CNN
 F 1 "+3.3V" H 8665 1673 50  0000 C CNN
 F 2 "" H 8650 1500 50  0001 C CNN
@@
 	8900 1950 9700 1950
 $Comp
-L power:+3.3V #PWR0119
+L power:+3.3V #PWR052
 U 1 1 61B19B18
 P 9950 3150
-F 0 "#PWR0119" H 9950 3000 50  0001 C CNN
+F 0 "#PWR052" H 9950 3000 50  0001 C CNN
 F 1 "+3.3V" H 9965 3323 50  0000 C CNN
 F 2 "" H 9950 3150 50  0001 C CNN
