File: KiCad-Project/ESP32/LEDDriver.sch (KiCad schematic (older format))
At the start: 2 parts, among them Q3 Q_NMOS_GDS, U5 TC4420CPA

Commit message: swap out 603 resistors for 805
Give us more room to work with if we have to fix something.
Changed lines of the file:
@@
 $Descr A4 11693 8268
 encoding utf-8
-Sheet 5 10
+Sheet 2 10
 Title ""
 Date ""
@@
 AR Path="/618EAA06/618FB99D" Ref="Q9"  Part="1"
 AR Path="/618EAB5C/618FB99D" Ref="Q10"  Part="1"
-F 0 "Q6" H 6054 3121 50  0000 L CNN
+F 0 "Q3" H 6054 3121 50  0000 L CNN
 F 1 "Q_NMOS_GDS" H 6054 3030 50  0000 L CNN
 F 2 "Package_TO_SOT_THT:TO-220-3_Vertical" H 6050 3175 50  0001 C CNN
@@
 AR Path="/618EAA06/6171033F" Ref="#PWR038"  Part="1"
 AR Path="/618EAB5C/6171033F" Ref="#PWR039"  Part="1"
-F 0 "#PWR035" H 4150 3675 50  0001 C CNN
+F 0 "#PWR039" H 4150 3675 50  0001 C CNN
 F 1 "GND" H 4155 3752 50  0000 C CNN
 F 2 "" H 4150 3925 50  0001 C CNN
@@
 AR Path="/618EAA06/618FB99C" Ref="U11"  Part="1"
 AR Path="/618EAB5C/618FB99C" Ref="U12"  Part="1"
-F 0 "U8" H 4375 3445 50  0000 C CNN
+F 0 "U5" H 4375 3445 50  0000 C CNN
 F 1 "TC4420CPA" H 4375 3354 50  0000 C CNN
 F 2 "TC4420CPA:DIP254P762X533-8" H 4375 2975 50  0001 L BNN
@@
 AR Path="/618EAA06/6188FB7C" Ref="#PWR0113"  Part="1"
 AR Path="/618EAB5C/6188FB7C" Ref="#PWR0115"  Part="1"
-F 0 "#PWR0107" H 5900 2000 50  0001 C CNN
+F 0 "#PWR0115" H 5900 2000 50  0001 C CNN
 F 1 "+24V" V 5915 2278 50  0000 L CNN
 F 2 "" H 5900 2150 50  0001 C CNN
@@
 AR Path="/618EAA06/618919ED" Ref="#PWR0114"  Part="1"
 AR Path="/618EAB5C/618919ED" Ref="#PWR0116"  Part="1"
-F 0 "#PWR0108" H 3375 2925 50  0001 C CNN
+F 0 "#PWR0116" H 3375 2925 50  0001 C CNN
 F 1 "+5V" V 3390 3203 50  0000 L CNN
 F 2 "" H 3375 3075 50  0001 C CNN

Commit message: Fixes in prep for printing
Making sure tolerance are in-spec for JLC PCB
Parts:
- Q3: MFG_PNUM (none) -> P30N06LE
Changed lines of the file:
@@
 $Descr A4 11693 8268
 encoding utf-8
-Sheet 2 10
+Sheet 6 10
 Title ""
 Date ""
@@
 AR Path="/618EAA06/618FB99D" Ref="Q9"  Part="1"
 AR Path="/618EAB5C/618FB99D" Ref="Q10"  Part="1"
-F 0 "Q3" H 6054 3121 50  0000 L CNN
+F 0 "Q7" H 6054 3121 50  0000 L CNN
 F 1 "Q_NMOS_GDS" H 6054 3030 50  0000 L CNN
 F 2 "Package_TO_SOT_THT:TO-220-3_Vertical" H 6050 3175 50  0001 C CNN
 F 3 "~" H 5850 3075 50  0001 C CNN
 F 4 "Mouser" H 5850 3075 50  0001 C CNN "SUPPLIER"
+F 5 "P30N06LE" H 5850 3075 50  0001 C CNN "MFG_PNUM"
 	1    5850 3075
 	1    0    0    -1
@@
 AR Path="/618EAA06/6171033F" Ref="#PWR038"  Part="1"
 AR Path="/618EAB5C/6171033F" Ref="#PWR039"  Part="1"
-F 0 "#PWR039" H 4150 3675 50  0001 C CNN
+F 0 "#PWR036" H 4150 3675 50  0001 C CNN
 F 1 "GND" H 4155 3752 50  0000 C CNN
 F 2 "" H 4150 3925 50  0001 C CNN
 F 3 "" H 4150 3925 50  0001 C CNN
 	1    4150 3925
-	1    0    0    -1
-$EndComp
-$Comp
-L TC4420CPA:TC4420CPA U?
-U 1 1 618FB99C
-P 4375 2975
-AR Path="/616EA041/618FB99C" Ref="U?"  Part="1"
-AR Path="/616F032A/618FB99C" Ref="U?"  Part="1"
-AR Path="/616F05F8/618FB99C" Ref="U?"  Part="1"
-AR Path="/616F41C8/618FB99C" Ref="U?"  Part="1"
-AR Path="/616F41CD/618FB99C" Ref="U?"  Part="1"
-AR Path="/616F41D2/618FB99C" Ref="U?"  Part="1"
-AR Path="/618E5B4E/618FB99C" Ref="U5"  Part="1"
-AR Path="/618E98F2/618FB99C" Ref="U?"  Part="1"
-AR Path="/618E9B79/618FB99C" Ref="U?"  Part="1"
-AR Path="/618E9C7A/618FB99C" Ref="U?"  Part="1"
-AR Path="/618E9DCB/618FB99C" Ref="U?"  Part="1"
-AR Path="/618E9EF4/618FB99C" Ref="U?"  Part="1"
-AR Path="/618EA306/618FB99C" Ref="U6"  Part="1"
-AR Path="/618EA5C6/618FB99C" Ref="U7"  Part="1"
-AR Path="/618EA73A/618FB99C" Ref="U8"  Part="1"
-AR Path="/618EA868/618FB99C" Ref="U9"  Part="1"
-AR Path="/618EA9C3/618FB99C" Ref="U10"  Part="1"
-AR Path="/618EAA06/618FB99C" Ref="U11"  Part="1"
-AR Path="/618EAB5C/618FB99C" Ref="U12"  Part="1"
-F 0 "U5" H 4375 3445 50  0000 C CNN
-F 1 "TC4420CPA" H 4375 3354 50  0000 C CNN
-F 2 "TC4420CPA:DIP254P762X533-8" H 4375 2975 50  0001 L BNN
-F 3 "" H 4375 2975 50  0001 L BNN
-F 4 "9762566" H 4375 2975 50  0001 L BNN "OC_FARNELL"
-F 5 "TC4420CPA" H 4375 2975 50  0001 L BNN "MPN"
-F 6 "DIP8" H 4375 2975 50  0001 L BNN "PACKAGE"
-F 7 "61K3536" H 4375 2975 50  0001 L BNN "OC_NEWARK"
-F 8 "Mouser" H 4375 2975 50  0001 L BNN "SUPPLIER"
-F 9 "TC4420CPA" H 4375 2975 50  0001 C CNN "MFG_PNUM"
-	1    4375 2975
 	1    0    0    -1
 $EndComp
@@
 AR Path="/618EAA06/6188FB7C" Ref="#PWR0113"  Part="1"
 AR Path="/618EAB5C/6188FB7C" Ref="#PWR0115"  Part="1"
-F 0 "#PWR0115" H 5900 2000 50  0001 C CNN
+F 0 "#PWR0109" H 5900 2000 50  0001 C CNN
 F 1 "+24V" V 5915 2278 50  0000 L CNN
 F 2 "" H 5900 2150 50  0001 C CNN
@@
 AR Path="/618EAA06/618919ED" Ref="#PWR0114"  Part="1"
 AR Path="/618EAB5C/618919ED" Ref="#PWR0116"  Part="1"
-F 0 "#PWR0116" H 3375 2925 50  0001 C CNN
+F 0 "#PWR0110" H 3375 2925 50  0001 C CNN
 F 1 "+5V" V 3390 3203 50  0000 L CNN
 F 2 "" H 3375 3075 50  0001 C CNN
@@
 Wire Wire Line
 	5900 2150 6100 2150
+$Comp
+L TC4420CPA:TC4420CPA U?
+U 1 1 618FB99C
+P 4375 2975
+AR Path="/616EA041/618FB99C" Ref="U?"  Part="1"
+AR Path="/616F032A/618FB99C" Ref="U?"  Part="1"
+AR Path="/616F05F8/618FB99C" Ref="U?"  Part="1"
+AR Path="/616F41C8/618FB99C" Ref="U?"  Part="1"
+AR Path="/616F41CD/618FB99C" Ref="U?"  Part="1"
+AR Path="/616F41D2/618FB99C" Ref="U?"  Part="1"
+AR Path="/618E5B4E/618FB99C" Ref="U5"  Part="1"
+AR Path="/618E98F2/618FB99C" Ref="U?"  Part="1"
+AR Path="/618E9B79/618FB99C" Ref="U?"  Part="1"
+AR Path="/618E9C7A/618FB99C" Ref="U?"  Part="1"
+AR Path="/618E9DCB/618FB99C" Ref="U?"  Part="1"
+AR Path="/618E9EF4/618FB99C" Ref="U?"  Part="1"
+AR Path="/618EA306/618FB99C" Ref="U6"  Part="1"
+AR Path="/618EA5C6/618FB99C" Ref="U7"  Part="1"
+AR Path="/618EA73A/618FB99C" Ref="U8"  Part="1"
+AR Path="/618EA868/618FB99C" Ref="U9"  Part="1"
+AR Path="/618EA9C3/618FB99C" Ref="U10"  Part="1"
+AR Path="/618EAA06/618FB99C" Ref="U11"  Part="1"
+AR Path="/618EAB5C/618FB99C" Ref="U12"  Part="1"
+F 0 "U9" H 4375 3445 50  0000 C CNN
+F 1 "TC4420CPA" H 4375 3354 50  0000 C CNN
+F 2 "TC4420CPA:DIP254P762X533-8" H 4375 2975 50  0001 L BNN
+F 3 "" H 4375 2975 50  0001 L BNN
+F 4 "9762566" H 4375 2975 50  0001 L BNN "OC_FARNELL"
+F 5 "TC4420CPA" H 4375 2975 50  0001 L BNN "MPN"
+F 6 "DIP8" H 4375 2975 50  0001 L BNN "PACKAGE"
+F 7 "61K3536" H 4375 2975 50  0001 L BNN "OC_NEWARK"
+F 8 "Mouser" H 4375 2975 50  0001 L BNN "SUPPLIER"
+F 9 "TC4420CPA" H 4375 2975 50  0001 C CNN "MFG_PNUM"
+	1    4375 2975
+	1    0    0    -1
+$EndComp
 $EndSCHEMATC

Commit message: Removed reverse voltage and increased size of power traces
Reverse voltage needed different components for 24 volt, and was a nice to have, so to keep cost down, opted to remove it.
Changed lines of the file:
@@
 $Descr A4 11693 8268
 encoding utf-8
-Sheet 6 10
+Sheet 8 10
 Title ""
 Date ""
@@
 AR Path="/618EAA06/618FB99D" Ref="Q9"  Part="1"
 AR Path="/618EAB5C/618FB99D" Ref="Q10"  Part="1"
-F 0 "Q7" H 6054 3121 50  0000 L CNN
+F 0 "Q10" H 6054 3121 50  0000 L CNN
 F 1 "Q_NMOS_GDS" H 6054 3030 50  0000 L CNN
 F 2 "Package_TO_SOT_THT:TO-220-3_Vertical" H 6050 3175 50  0001 C CNN
@@
 AR Path="/618EAA06/6171033F" Ref="#PWR038"  Part="1"
 AR Path="/618EAB5C/6171033F" Ref="#PWR039"  Part="1"
-F 0 "#PWR036" H 4150 3675 50  0001 C CNN
+F 0 "#PWR039" H 4150 3675 50  0001 C CNN
 F 1 "GND" H 4155 3752 50  0000 C CNN
 F 2 "" H 4150 3925 50  0001 C CNN
@@
 AR Path="/618EAA06/6188FB7C" Ref="#PWR0113"  Part="1"
 AR Path="/618EAB5C/6188FB7C" Ref="#PWR0115"  Part="1"
-F 0 "#PWR0109" H 5900 2000 50  0001 C CNN
+F 0 "#PWR0115" H 5900 2000 50  0001 C CNN
 F 1 "+24V" V 5915 2278 50  0000 L CNN
 F 2 "" H 5900 2150 50  0001 C CNN
@@
 AR Path="/618EAA06/618919ED" Ref="#PWR0114"  Part="1"
 AR Path="/618EAB5C/618919ED" Ref="#PWR0116"  Part="1"
-F 0 "#PWR0110" H 3375 2925 50  0001 C CNN
+F 0 "#PWR0116" H 3375 2925 50  0001 C CNN
 F 1 "+5V" V 3390 3203 50  0000 L CNN
 F 2 "" H 3375 3075 50  0001 C CNN
@@
 AR Path="/618EAA06/618FB99C" Ref="U11"  Part="1"
 AR Path="/618EAB5C/618FB99C" Ref="U12"  Part="1"
-F 0 "U9" H 4375 3445 50  0000 C CNN
+F 0 "U12" H 4375 3445 50  0000 C CNN
 F 1 "TC4420CPA" H 4375 3354 50  0000 C CNN
 F 2 "TC4420CPA:DIP254P762X533-8" H 4375 2975 50  0001 L BNN

Commit message: Move on board test LED to a better pin. and swap TX/RX UART pins
Changed lines of the file:
@@
 $Descr A4 11693 8268
 encoding utf-8
-Sheet 8 10
+Sheet 5 10
 Title ""
 Date ""
@@
 AR Path="/618EAA06/618FB99D" Ref="Q9"  Part="1"
 AR Path="/618EAB5C/618FB99D" Ref="Q10"  Part="1"
-F 0 "Q10" H 6054 3121 50  0000 L CNN
+F 0 "Q6" H 6054 3121 50  0000 L CNN
 F 1 "Q_NMOS_GDS" H 6054 3030 50  0000 L CNN
 F 2 "Package_TO_SOT_THT:TO-220-3_Vertical" H 6050 3175 50  0001 C CNN
@@
 AR Path="/618EAA06/6171033F" Ref="#PWR038"  Part="1"
 AR Path="/618EAB5C/6171033F" Ref="#PWR039"  Part="1"
-F 0 "#PWR039" H 4150 3675 50  0001 C CNN
+F 0 "#PWR035" H 4150 3675 50  0001 C CNN
 F 1 "GND" H 4155 3752 50  0000 C CNN
 F 2 "" H 4150 3925 50  0001 C CNN
@@
 AR Path="/618EAA06/6188FB7C" Ref="#PWR0113"  Part="1"
 AR Path="/618EAB5C/6188FB7C" Ref="#PWR0115"  Part="1"
-F 0 "#PWR0115" H 5900 2000 50  0001 C CNN
+F 0 "#PWR0107" H 5900 2000 50  0001 C CNN
 F 1 "+24V" V 5915 2278 50  0000 L CNN
 F 2 "" H 5900 2150 50  0001 C CNN
@@
 AR Path="/618EAA06/618919ED" Ref="#PWR0114"  Part="1"
 AR Path="/618EAB5C/618919ED" Ref="#PWR0116"  Part="1"
-F 0 "#PWR0116" H 3375 2925 50  0001 C CNN
+F 0 "#PWR0108" H 3375 2925 50  0001 C CNN
 F 1 "+5V" V 3390 3203 50  0000 L CNN
 F 2 "" H 3375 3075 50  0001 C CNN
@@
 AR Path="/618EAA06/618FB99C" Ref="U11"  Part="1"
 AR Path="/618EAB5C/618FB99C" Ref="U12"  Part="1"
-F 0 "U12" H 4375 3445 50  0000 C CNN
+F 0 "U8" H 4375 3445 50  0000 C CNN
 F 1 "TC4420CPA" H 4375 3354 50  0000 C CNN
 F 2 "TC4420CPA:DIP254P762X533-8" H 4375 2975 50  0001 L BNN

Commit message: Aligning parts to each other
Parts:
- added JP3: Driver Bypass, symbol Jumper:SolderJumper_2_Open
Connections:
- net SIG: now also JP3.1 (A)
- net at Q3.1 (G), U5.7 (OUTPUT): now also JP3.2 (B)
Changed lines of the file:
@@
 $Descr A4 11693 8268
 encoding utf-8
-Sheet 5 10
+Sheet 2 10
 Title ""
 Date ""
@@
 LED-
 Wire Wire Line
-	3425 2875 3575 2875
+	3425 2875 3500 2875
 Wire Wire Line
 	5950 2875 6100 2875
@@
 AR Path="/618EAA06/618FB99D" Ref="Q9"  Part="1"
 AR Path="/618EAB5C/618FB99D" Ref="Q10"  Part="1"
-F 0 "Q6" H 6054 3121 50  0000 L CNN
+F 0 "Q3" H 6054 3121 50  0000 L CNN
 F 1 "Q_NMOS_GDS" H 6054 3030 50  0000 L CNN
 F 2 "Package_TO_SOT_THT:TO-220-3_Vertical" H 6050 3175 50  0001 C CNN
@@
 AR Path="/618EAA06/6171033F" Ref="#PWR038"  Part="1"
 AR Path="/618EAB5C/6171033F" Ref="#PWR039"  Part="1"
-F 0 "#PWR035" H 4150 3675 50  0001 C CNN
+F 0 "#PWR032" H 4150 3675 50  0001 C CNN
 F 1 "GND" H 4155 3752 50  0000 C CNN
 F 2 "" H 4150 3925 50  0001 C CNN
@@
 AR Path="/618EAA06/6188FB7C" Ref="#PWR0113"  Part="1"
 AR Path="/618EAB5C/6188FB7C" Ref="#PWR0115"  Part="1"
-F 0 "#PWR0107" H 5900 2000 50  0001 C CNN
+F 0 "#PWR0101" H 5900 2000 50  0001 C CNN
 F 1 "+24V" V 5915 2278 50  0000 L CNN
 F 2 "" H 5900 2150 50  0001 C CNN
@@
 AR Path="/618EAA06/618919ED" Ref="#PWR0114"  Part="1"
 AR Path="/618EAB5C/618919ED" Ref="#PWR0116"  Part="1"
-F 0 "#PWR0108" H 3375 2925 50  0001 C CNN
+F 0 "#PWR0102" H 3375 2925 50  0001 C CNN
 F 1 "+5V" V 3390 3203 50  0000 L CNN
 F 2 "" H 3375 3075 50  0001 C CNN
@@
 	3500 3075 3575 3075
 Wire Wire Line
-	5175 3075 5650 3075
+	5175 3075 5425 3075
 NoConn ~ 5175 3175
 Wire Wire Line
@@
 AR Path="/618EAA06/618FB99C" Ref="U11"  Part="1"
 AR Path="/618EAB5C/618FB99C" Ref="U12"  Part="1"
-F 0 "U8" H 4375 3445 50  0000 C CNN
+F 0 "U5" H 4375 3445 50  0000 C CNN
 F 1 "TC4420CPA" H 4375 3354 50  0000 C CNN
 F 2 "TC4420CPA:DIP254P762X533-8" H 4375 2975 50  0001 L BNN
@@
 	1    0    0    -1
 $EndComp
+$Comp
+L Jumper:SolderJumper_2_Open JP3
+U 1 1 61AE4A33
+P 4525 2300
+AR Path="/618E5B4E/61AE4A33" Ref="JP3"  Part="1"
+AR Path="/618EA306/61AE4A33" Ref="JP4"  Part="1"
+AR Path="/618EA5C6/61AE4A33" Ref="JP5"  Part="1"
+AR Path="/618EA73A/61AE4A33" Ref="JP6"  Part="1"
+AR Path="/618EA868/61AE4A33" Ref="JP7"  Part="1"
+AR Path="/618EA9C3/61AE4A33" Ref="JP8"  Part="1"
+AR Path="/618EAA06/61AE4A33" Ref="JP9"  Part="1"
+AR Path="/618EAB5C/61AE4A33" Ref="JP10"  Part="1"
+F 0 "JP3" H 4525 2505 50  0000 C CNN
+F 1 "Driver Bypass" H 4525 2414 50  0000 C CNN
+F 2 "" H 4525 2300 50  0001 C CNN
+F 3 "~" H 4525 2300 50  0001 C CNN
+	1    4525 2300
+	1    0    0    -1
+$EndComp
+Wire Wire Line
+	3500 2875 3500 2300
+Wire Wire Line
+	3500 2300 4375 2300
+Connection ~ 3500 2875
+Wire Wire Line
+	3500 2875 3575 2875
+Wire Wire Line
+	4675 2300 5425 2300
+Wire Wire Line
+	5425 2300 5425 3075
+Connection ~ 5425 3075
+Wire Wire Line
+	5425 3075 5650 3075
 $EndSCHEMATC

Commit message: update pin labels
Parts:
- JP3: footprint (none) -> Jumper:SolderJumper-2_P1.3mm_Open_RoundedPad1.0x1.5mm
- Q3: value Q_NMOS_GDS -> P30N06LE
Changed lines of the file:
@@
 AR Path="/618EAB5C/618FB99D" Ref="Q10"  Part="1"
 F 0 "Q3" H 6054 3121 50  0000 L CNN
-F 1 "Q_NMOS_GDS" H 6054 3030 50  0000 L CNN
+F 1 "P30N06LE" H 6054 3030 50  0000 L CNN
 F 2 "Package_TO_SOT_THT:TO-220-3_Vertical" H 6050 3175 50  0001 C CNN
 F 3 "~" H 5850 3075 50  0001 C CNN
@@
 F 0 "JP3" H 4525 2505 50  0000 C CNN
 F 1 "Driver Bypass" H 4525 2414 50  0000 C CNN
-F 2 "" H 4525 2300 50  0001 C CNN
+F 2 "Jumper:SolderJumper-2_P1.3mm_Open_RoundedPad1.0x1.5mm" H 4525 2300 50  0001 C CNN
 F 3 "~" H 4525 2300 50  0001 C CNN
 	1    4525 2300
