File: KiCad-Project/ESP32/LEDDriver.sch (KiCad schematic (older format))
At the start: 3 parts, among them Q3 P30N06LE, U5 TC4420CPA

Commit message: Reset annotations
Parts:
- renumbered JP3 to JP1, Q3 to Q1, U5 to U3
Changed lines of the file:
@@
 AR Path="/616F41CD/618FB99D" Ref="Q?"  Part="1"
 AR Path="/616F41D2/618FB99D" Ref="Q?"  Part="1"
-AR Path="/618E5B4E/618FB99D" Ref="Q3"  Part="1"
+AR Path="/618E5B4E/618FB99D" Ref="Q1"  Part="1"
 AR Path="/618E98F2/618FB99D" Ref="Q?"  Part="1"
 AR Path="/618E9B79/618FB99D" Ref="Q?"  Part="1"
@@
 AR Path="/618E9DCB/618FB99D" Ref="Q?"  Part="1"
 AR Path="/618E9EF4/618FB99D" Ref="Q?"  Part="1"
-AR Path="/618EA306/618FB99D" Ref="Q4"  Part="1"
-AR Path="/618EA5C6/618FB99D" Ref="Q5"  Part="1"
-AR Path="/618EA73A/618FB99D" Ref="Q6"  Part="1"
-AR Path="/618EA868/618FB99D" Ref="Q7"  Part="1"
-AR Path="/618EA9C3/618FB99D" Ref="Q8"  Part="1"
-AR Path="/618EAA06/618FB99D" Ref="Q9"  Part="1"
-AR Path="/618EAB5C/618FB99D" Ref="Q10"  Part="1"
-F 0 "Q3" H 6054 3121 50  0000 L CNN
+AR Path="/618EA306/618FB99D" Ref="Q2"  Part="1"
+AR Path="/618EA5C6/618FB99D" Ref="Q3"  Part="1"
+AR Path="/618EA73A/618FB99D" Ref="Q4"  Part="1"
+AR Path="/618EA868/618FB99D" Ref="Q5"  Part="1"
+AR Path="/618EA9C3/618FB99D" Ref="Q6"  Part="1"
+AR Path="/618EAA06/618FB99D" Ref="Q7"  Part="1"
+AR Path="/618EAB5C/618FB99D" Ref="Q8"  Part="1"
+F 0 "Q8" H 6054 3121 50  0000 L CNN
 F 1 "P30N06LE" H 6054 3030 50  0000 L CNN
 F 2 "Package_TO_SOT_THT:TO-220-3_Vertical" H 6050 3175 50  0001 C CNN
@@
 AR Path="/616F41CD/6171033F" Ref="#PWR?"  Part="1"
 AR Path="/616F41D2/6171033F" Ref="#PWR?"  Part="1"
-AR Path="/618E5B4E/6171033F" Ref="#PWR032"  Part="1"
+AR Path="/618E5B4E/6171033F" Ref="#PWR015"  Part="1"
 AR Path="/618E98F2/6171033F" Ref="#PWR?"  Part="1"
 AR Path="/618E9B79/6171033F" Ref="#PWR?"  Part="1"
@@
 AR Path="/618E9DCB/6171033F" Ref="#PWR?"  Part="1"
 AR Path="/618E9EF4/6171033F" Ref="#PWR?"  Part="1"
-AR Path="/618EA306/6171033F" Ref="#PWR033"  Part="1"
-AR Path="/618EA5C6/6171033F" Ref="#PWR034"  Part="1"
-AR Path="/618EA73A/6171033F" Ref="#PWR035"  Part="1"
-AR Path="/618EA868/6171033F" Ref="#PWR036"  Part="1"
-AR Path="/618EA9C3/6171033F" Ref="#PWR037"  Part="1"
-AR Path="/618EAA06/6171033F" Ref="#PWR038"  Part="1"
-AR Path="/618EAB5C/6171033F" Ref="#PWR039"  Part="1"
-F 0 "#PWR032" H 4150 3675 50  0001 C CNN
+AR Path="/618EA306/6171033F" Ref="#PWR018"  Part="1"
+AR Path="/618EA5C6/6171033F" Ref="#PWR021"  Part="1"
+AR Path="/618EA73A/6171033F" Ref="#PWR024"  Part="1"
+AR Path="/618EA868/6171033F" Ref="#PWR027"  Part="1"
+AR Path="/618EA9C3/6171033F" Ref="#PWR030"  Part="1"
+AR Path="/618EAA06/6171033F" Ref="#PWR033"  Part="1"
+AR Path="/618EAB5C/6171033F" Ref="#PWR036"  Part="1"
+F 0 "#PWR036" H 4150 3675 50  0001 C CNN
 F 1 "GND" H 4155 3752 50  0000 C CNN
 F 2 "" H 4150 3925 50  0001 C CNN
@@
 	3375 3075 3500 3075
 $Comp
-L power:+24V #PWR0105
+L power:+24V #PWR022
 U 1 1 6188FB7C
 P 5900 2150
-AR Path="/618EA5C6/6188FB7C" Ref="#PWR0105"  Part="1"
-AR Path="/618E5B4E/6188FB7C" Ref="#PWR0101"  Part="1"
-AR Path="/618EA306/6188FB7C" Ref="#PWR0103"  Part="1"
-AR Path="/618EA73A/6188FB7C" Ref="#PWR0107"  Part="1"
-AR Path="/618EA868/6188FB7C" Ref="#PWR0109"  Part="1"
-AR Path="/618EA9C3/6188FB7C" Ref="#PWR0111"  Part="1"
-AR Path="/618EAA06/6188FB7C" Ref="#PWR0113"  Part="1"
-AR Path="/618EAB5C/6188FB7C" Ref="#PWR0115"  Part="1"
-F 0 "#PWR0101" H 5900 2000 50  0001 C CNN
+AR Path="/618EA5C6/6188FB7C" Ref="#PWR022"  Part="1"
+AR Path="/618E5B4E/6188FB7C" Ref="#PWR016"  Part="1"
+AR Path="/618EA306/6188FB7C" Ref="#PWR019"  Part="1"
+AR Path="/618EA73A/6188FB7C" Ref="#PWR025"  Part="1"
+AR Path="/618EA868/6188FB7C" Ref="#PWR028"  Part="1"
+AR Path="/618EA9C3/6188FB7C" Ref="#PWR031"  Part="1"
+AR Path="/618EAA06/6188FB7C" Ref="#PWR034"  Part="1"
+AR Path="/618EAB5C/6188FB7C" Ref="#PWR037"  Part="1"
+F 0 "#PWR037" H 5900 2000 50  0001 C CNN
 F 1 "+24V" V 5915 2278 50  0000 L CNN
 F 2 "" H 5900 2150 50  0001 C CNN
@@
 $EndComp
 $Comp
-L power:+5V #PWR0106
+L power:+5V #PWR020
 U 1 1 618919ED
 P 3375 3075
-AR Path="/618EA5C6/618919ED" Ref="#PWR0106"  Part="1"
-AR Path="/618E5B4E/618919ED" Ref="#PWR0102"  Part="1"
-AR Path="/618EA306/618919ED" Ref="#PWR0104"  Part="1"
-AR Path="/618EA73A/618919ED" Ref="#PWR0108"  Part="1"
-AR Path="/618EA868/618919ED" Ref="#PWR0110"  Part="1"
-AR Path="/618EA9C3/618919ED" Ref="#PWR0112"  Part="1"
-AR Path="/618EAA06/618919ED" Ref="#PWR0114"  Part="1"
-AR Path="/618EAB5C/618919ED" Ref="#PWR0116"  Part="1"
-F 0 "#PWR0102" H 3375 2925 50  0001 C CNN
+AR Path="/618EA5C6/618919ED" Ref="#PWR020"  Part="1"
+AR Path="/618E5B4E/618919ED" Ref="#PWR014"  Part="1"
+AR Path="/618EA306/618919ED" Ref="#PWR017"  Part="1"
+AR Path="/618EA73A/618919ED" Ref="#PWR023"  Part="1"
+AR Path="/618EA868/618919ED" Ref="#PWR026"  Part="1"
+AR Path="/618EA9C3/618919ED" Ref="#PWR029"  Part="1"
+AR Path="/618EAA06/618919ED" Ref="#PWR032"  Part="1"
+AR Path="/618EAB5C/618919ED" Ref="#PWR035"  Part="1"
+F 0 "#PWR035" H 3375 2925 50  0001 C CNN
 F 1 "+5V" V 3390 3203 50  0000 L CNN
 F 2 "" H 3375 3075 50  0001 C CNN
@@
 AR Path="/616F41CD/618FB99C" Ref="U?"  Part="1"
 AR Path="/616F41D2/618FB99C" Ref="U?"  Part="1"
-AR Path="/618E5B4E/618FB99C" Ref="U5"  Part="1"
+AR Path="/618E5B4E/618FB99C" Ref="U3"  Part="1"
 AR Path="/618E98F2/618FB99C" Ref="U?"  Part="1"
 AR Path="/618E9B79/618FB99C" Ref="U?"  Part="1"
@@
 AR Path="/618E9DCB/618FB99C" Ref="U?"  Part="1"
 AR Path="/618E9EF4/618FB99C" Ref="U?"  Part="1"
-AR Path="/618EA306/618FB99C" Ref="U6"  Part="1"
-AR Path="/618EA5C6/618FB99C" Ref="U7"  Part="1"
-AR Path="/618EA73A/618FB99C" Ref="U8"  Part="1"
-AR Path="/618EA868/618FB99C" Ref="U9"  Part="1"
-AR Path="/618EA9C3/618FB99C" Ref="U10"  Part="1"
-AR Path="/618EAA06/618FB99C" Ref="U11"  Part="1"
-AR Path="/618EAB5C/618FB99C" Ref="U12"  Part="1"
-F 0 "U5" H 4375 3445 50  0000 C CNN
+AR Path="/618EA306/618FB99C" Ref="U4"  Part="1"
+AR Path="/618EA5C6/618FB99C" Ref="U5"  Part="1"
+AR Path="/618EA73A/618FB99C" Ref="U6"  Part="1"
+AR Path="/618EA868/618FB99C" Ref="U7"  Part="1"
+AR Path="/618EA9C3/618FB99C" Ref="U8"  Part="1"
+AR Path="/618EAA06/618FB99C" Ref="U9"  Part="1"
+AR Path="/618EAB5C/618FB99C" Ref="U10"  Part="1"
+F 0 "U10" H 4375 3445 50  0000 C CNN
 F 1 "TC4420CPA" H 4375 3354 50  0000 C CNN
 F 2 "TC4420CPA:DIP254P762X533-8" H 4375 2975 50  0001 L BNN
@@
 $EndComp
 $Comp
-L Jumper:SolderJumper_2_Open JP3
+L Jumper:SolderJumper_2_Open JP1
 U 1 1 61AE4A33
 P 4525 2300
-AR Path="/618E5B4E/61AE4A33" Ref="JP3"  Part="1"
-AR Path="/618EA306/61AE4A33" Ref="JP4"  Part="1"
-AR Path="/618EA5C6/61AE4A33" Ref="JP5"  Part="1"
-AR Path="/618EA73A/61AE4A33" Ref="JP6"  Part="1"
-AR Path="/618EA868/61AE4A33" Ref="JP7"  Part="1"
-AR Path="/618EA9C3/61AE4A33" Ref="JP8"  Part="1"
-AR Path="/618EAA06/61AE4A33" Ref="JP9"  Part="1"
-AR Path="/618EAB5C/61AE4A33" Ref="JP10"  Part="1"
-F 0 "JP3" H 4525 2505 50  0000 C CNN
+AR Path="/618E5B4E/61AE4A33" Ref="JP1"  Part="1"
+AR Path="/618EA306/61AE4A33" Ref="JP2"  Part="1"
+AR Path="/618EA5C6/61AE4A33" Ref="JP3"  Part="1"
+AR Path="/618EA73A/61AE4A33" Ref="JP4"  Part="1"
+AR Path="/618EA868/61AE4A33" Ref="JP5"  Part="1"
+AR Path="/618EA9C3/61AE4A33" Ref="JP6"  Part="1"
+AR Path="/618EAA06/61AE4A33" Ref="JP7"  Part="1"
+AR Path="/618EAB5C/61AE4A33" Ref="JP8"  Part="1"
+F 0 "JP8" H 4525 2505 50  0000 C CNN
 F 1 "Driver Bypass" H 4525 2414 50  0000 C CNN
 F 2 "Jumper:SolderJumper-2_P1.3mm_Open_RoundedPad1.0x1.5mm" H 4525 2300 50  0001 C CNN
