File: KiCad-Project/ESP32/ESP32LedDriverV2.sch (KiCad schematic (older format))
At the start: 20 parts, among them J1 Power, J2 LED Terminal, U1 INA219AxD, U2 R-78C5.0-1.0

Commit message: Reset annotations
Parts:
- U1: renamed from U2; Alt (none) -> MDS06F-05
- renumbered C3 to C1, C1 to C3, D2 to D1, R3 to R1, R4 to R2, R5 to R3, R6 to R4, R7 to R5, U1 to U2
Other:
- moved on the sheet: H1, H2, H3, H4
Changed lines of the file:
@@
 Z8
 $Comp
-L Regulator_Switching:R-78C5.0-1.0 U2
+L Regulator_Switching:R-78C5.0-1.0 U1
 U 1 1 6166B921
 P 2150 6900
-F 0 "U2" H 2150 7142 50  0000 C CNN
+F 0 "U1" H 2150 7142 50  0000 C CNN
 F 1 "R-78C5.0-1.0" H 2150 7051 50  0000 C CNN
 F 2 "Converter_DCDC:Converter_DCDC_RECOM_R-78E-0.5_THT" H 2200 6650 50  0001 L CIN
@@
 F 4 "R-78C5.0-1.0" H 2150 6900 50  0001 C CNN "MFG_PNUM"
 F 5 "Mouser" H 2150 6900 50  0001 C CNN "SUPPLIER"
+F 6 "MDS06F-05" H 2150 6900 50  0001 C CNN "Alt"
 	1    2150 6900
 	1    0    0    -1
 $EndComp
 $Comp
-L power:GND #PWR08
+L power:GND #PWR07
 U 1 1 616719E7
 P 2150 7375
-F 0 "#PWR08" H 2150 7125 50  0001 C CNN
+F 0 "#PWR07" H 2150 7125 50  0001 C CNN
 F 1 "GND" H 2155 7202 50  0000 C CNN
 F 2 "" H 2150 7375 50  0001 C CNN
@@
 	2450 6900 2525 6900
 $Comp
-L Device:CP1 C3
+L Device:CP1 C1
 U 1 1 618025B0
 P 1550 7150
-F 0 "C3" H 1665 7196 50  0000 L CNN
+F 0 "C1" H 1665 7196 50  0000 L CNN
 F 1 "330uF" H 1665 7105 50  0000 L CNN
 F 2 "Capacitor_THT:CP_Radial_D8.0mm_P3.50mm" H 1550 7150 50  0001 C CNN
@@
 $EndComp
 $Comp
-L Analog_ADC:INA219AxD U1
+L Analog_ADC:INA219AxD U2
 U 1 1 61975DF1
 P 2400 4825
-F 0 "U1" H 2175 5175 50  0000 C CNN
+F 0 "U2" H 2175 5175 50  0000 C CNN
 F 1 "INA219AxD" H 2675 4450 50  0000 C CNN
 F 2 "Package_SO:SOIC-8_3.9x4.9mm_P1.27mm" H 3200 4475 50  0001 C CNN
@@
 	1925 4925 2000 4925
 $Comp
-L power:+5V #PWR010
+L power:+5V #PWR011
 U 1 1 61987470
 P 3175 6900
-F 0 "#PWR010" H 3175 6750 50  0001 C CNN
+F 0 "#PWR011" H 3175 6750 50  0001 C CNN
 F 1 "+5V" V 3190 7028 50  0000 L CNN
 F 2 "" H 3175 6900 50  0001 C CNN
@@
 $EndComp
 $Comp
-L power:GND #PWR07
+L power:GND #PWR09
 U 1 1 61988340
 P 2400 5300
-F 0 "#PWR07" H 2400 5050 50  0001 C CNN
+F 0 "#PWR09" H 2400 5050 50  0001 C CNN
 F 1 "GND" H 2405 5127 50  0000 C CNN
 F 2 "" H 2400 5300 50  0001 C CNN
@@
 	2400 5225 2400 5300
 $Comp
-L power:+24V #PWR06
+L power:+24V #PWR03
 U 1 1 61997EB9
 P 1450 6900
-F 0 "#PWR06" H 1450 6750 50  0001 C CNN
+F 0 "#PWR03" H 1450 6750 50  0001 C CNN
 F 1 "+24V" H 1465 7073 50  0000 C CNN
 F 2 "" H 1450 6900 50  0001 C CNN
@@
 	2950 4200 2950 4100
 $Comp
-L Device:R_US R5
+L Device:R_US R3
 U 1 1 619C7D5F
 P 3325 4350
-F 0 "R5" H 3393 4396 50  0000 L CNN
+F 0 "R3" H 3393 4396 50  0000 L CNN
 F 1 "10K" H 3393 4305 50  0000 L CNN
 F 2 "Resistor_SMD:R_0805_2012Metric" V 3365 4340 50  0001 C CNN
@@
 $EndComp
 $Comp
-L Device:R_US R4
+L Device:R_US R2
 U 1 1 619C6847
 P 2950 4350
-F 0 "R4" H 3018 4396 50  0000 L CNN
+F 0 "R2" H 3018 4396 50  0000 L CNN
 F 1 "10K" H 3018 4305 50  0000 L CNN
 F 2 "Resistor_SMD:R_0805_2012Metric" V 2990 4340 50  0001 C CNN
@@
 $EndComp
 $Comp
-L power:+3.3V #PWR09
+L power:+3.3V #PWR010
 U 1 1 6198BC0D
 P 3125 3975
-F 0 "#PWR09" H 3125 3825 50  0001 C CNN
+F 0 "#PWR010" H 3125 3825 50  0001 C CNN
 F 1 "+3.3V" H 3140 4148 50  0000 C CNN
 F 2 "" H 3125 3975 50  0001 C CNN
@@
 Connection ~ 3325 4725
 $Comp
-L power:+3.3V #PWR011
+L power:+3.3V #PWR013
 U 1 1 619FB409
 P 3725 5100
-F 0 "#PWR011" H 3725 4950 50  0001 C CNN
+F 0 "#PWR013" H 3725 4950 50  0001 C CNN
 F 1 "+3.3V" V 3725 5325 50  0000 C CNN
 F 2 "" H 3725 5100 50  0001 C CNN
@@
 $EndComp
 $Comp
-L Device:R_US R6
+L Device:R_US R4
 U 1 1 619FB40F
 P 3350 4925
-F 0 "R6" V 3250 4875 50  0000 L CNN
+F 0 "R4" V 3250 4875 50  0000 L CNN
 F 1 "10K" V 3418 4880 50  0000 L CNN
 F 2 "Resistor_SMD:R_0805_2012Metric" V 3390 4915 50  0001 C CNN
@@
 	3600 5100 3725 5100
 $Comp
-L Device:R_US R7
+L Device:R_US R5
 U 1 1 619FB418
 P 3350 5225
-F 0 "R7" V 3250 5175 50  0000 L CNN
+F 0 "R5" V 3250 5175 50  0000 L CNN
 F 1 "10K" V 3418 5180 50  0000 L CNN
 F 2 "Resistor_SMD:R_0805_2012Metric" V 3390 5215 50  0001 C CNN
@@
 	3000 5025 3000 5225
 $Comp
-L Device:R_US R3
+L Device:R_US R1
 U 1 1 61A04746
 P 1325 5350
-F 0 "R3" V 1225 5300 50  0000 L CNN
+F 0 "R1" V 1225 5300 50  0000 L CNN
 F 1 "0.1Ω 1% 1W" H 1375 5375 50  0000 L CNN
 F 2 "Resistor_SMD:R_2512_6332Metric" V 1365 5340 50  0001 C CNN
@@
 L Mechanical:MountingHole H2
 U 1 1 618FF15C
-P 5525 7375
-F 0 "H2" H 5625 7421 50  0000 L CNN
-F 1 "MountingHole" H 5625 7330 50  0000 L CNN
-F 2 "MountingHole:MountingHole_3.2mm_M3" H 5525 7375 50  0001 C CNN
-F 3 "~" H 5525 7375 50  0001 C CNN
-	1    5525 7375
+P 5550 7400
+F 0 "H2" H 5650 7446 50  0000 L CNN
+F 1 "MountingHole" H 5650 7355 50  0000 L CNN
+F 2 "MountingHole:MountingHole_3.2mm_M3" H 5550 7400 50  0001 C CNN
+F 3 "~" H 5550 7400 50  0001 C CNN
+	1    5550 7400
 	1    0    0    -1
 $EndComp
@@
 L Mechanical:MountingHole H1
 U 1 1 618FF92E
-P 5525 7175
-F 0 "H1" H 5625 7221 50  0000 L CNN
-F 1 "MountingHole" H 5625 7130 50  0000 L CNN
-F 2 "MountingHole:MountingHole_3.2mm_M3" H 5525 7175 50  0001 C CNN
-F 3 "~" H 5525 7175 50  0001 C CNN
-	1    5525 7175
+P 5550 7200
+F 0 "H1" H 5650 7246 50  0000 L CNN
+F 1 "MountingHole" H 5650 7155 50  0000 L CNN
+F 2 "MountingHole:MountingHole_3.2mm_M3" H 5550 7200 50  0001 C CNN
+F 3 "~" H 5550 7200 50  0001 C CNN
+	1    5550 7200
 	1    0    0    -1
 $EndComp
@@
 L Mechanical:MountingHole H3
 U 1 1 619003B7
-P 5525 7600
-F 0 "H3" H 5625 7646 50  0000 L CNN
-F 1 "MountingHole" H 5625 7555 50  0000 L CNN
-F 2 "MountingHole:MountingHole_3.2mm_M3" H 5525 7600 50  0001 C CNN
-F 3 "~" H 5525 7600 50  0001 C CNN
-	1    5525 7600
+P 5550 7625
+F 0 "H3" H 5650 7671 50  0000 L CNN
+F 1 "MountingHole" H 5650 7580 50  0000 L CNN
+F 2 "MountingHole:MountingHole_3.2mm_M3" H 5550 7625 50  0001 C CNN
+F 3 "~" H 5550 7625 50  0001 C CNN
+	1    5550 7625
 	1    0    0    -1
 $EndComp
@@
 L Mechanical:MountingHole H4
 U 1 1 6191D5BF
-P 5550 7825
-F 0 "H4" H 5650 7871 50  0000 L CNN
-F 1 "MountingHole" H 5650 7780 50  0000 L CNN
-F 2 "MountingHole:MountingHole_3.2mm_M3" H 5550 7825 50  0001 C CNN
-F 3 "~" H 5550 7825 50  0001 C CNN
-	1    5550 7825
+P 5575 7850
+F 0 "H4" H 5675 7896 50  0000 L CNN
+F 1 "MountingHole" H 5675 7805 50  0000 L CNN
+F 2 "MountingHole:MountingHole_3.2mm_M3" H 5575 7850 50  0001 C CNN
+F 3 "~" H 5575 7850 50  0001 C CNN
+	1    5575 7850
 	1    0    0    -1
 $EndComp
@@
 	1450 2775 1450 2700
 $Comp
-L Device:D_Zener D2
+L Device:D_Zener D1
 U 1 1 6188BA26
 P 1450 2925
-F 0 "D2" V 1404 3005 50  0000 L CNN
+F 0 "D1" V 1404 3005 50  0000 L CNN
 F 1 "D_Zener 25v" V 1495 3005 50  0000 L CNN
 F 2 "Diode_THT:D_DO-35_SOD27_P7.62mm_Horizontal" H 1450 2925 50  0001 C CNN
@@
 Connection ~ 2400 2700
 $Comp
-L power:GND #PWR03
+L power:GND #PWR08
 U 1 1 6188B470
 P 2400 3125
-F 0 "#PWR03" H 2400 2875 50  0001 C CNN
+F 0 "#PWR08" H 2400 2875 50  0001 C CNN
 F 1 "GND" H 2405 2952 50  0000 C CNN
 F 2 "" H 2400 3125 50  0001 C CNN
@@
 $EndComp
 $Comp
-L Device:C C1
+L Device:C C3
 U 1 1 6186C17D
 P 2400 2850
-F 0 "C1" H 2515 2896 50  0000 L CNN
+F 0 "C3" H 2515 2896 50  0000 L CNN
 F 1 "100uF" H 2515 2805 50  0000 L CNN
 F 2 "Capacitor_THT:CP_Radial_D5.0mm_P2.00mm" H 2438 2700 50  0001 C CNN
@@
 	1550 6900 1850 6900
 $Comp
-L power:+24V #PWR0117
+L power:+24V #PWR06
 U 1 1 619E5019
 P 1875 5725
-F 0 "#PWR0117" H 1875 5575 50  0001 C CNN
+F 0 "#PWR06" H 1875 5575 50  0001 C CNN
 F 1 "+24V" H 1890 5898 50  0000 C CNN
 F 2 "" H 1875 5725 50  0001 C CNN
@@
 $EndSheet
 $Comp
-L power:PWR_FLAG #FLG0111
+L power:PWR_FLAG #FLG01
 U 1 1 61941C7D
 P 1325 1425
-F 0 "#FLG0111" H 1325 1500 50  0001 C CNN
+F 0 "#FLG01" H 1325 1500 50  0001 C CNN
 F 1 "PWR_FLAG" H 1150 1575 50  0000 C CNN
 F 2 "" H 1325 1425 50  0001 C CNN
@@
 	3600 4925 3600 5100
 $Comp
-L power:GND #PWR0118
+L power:GND #PWR012
 U 1 1 6194D52A
 P 3325 1500
-F 0 "#PWR0118" H 3325 1250 50  0001 C CNN
+F 0 "#PWR012" H 3325 1250 50  0001 C CNN
 F 1 "GND" V 3330 1372 50  0000 R CNN
 F 2 "" H 3325 1500 50  0001 C CNN
@@
 	3325 1500 3325 1300
 $Comp
-L power:PWR_FLAG #FLG0102
+L power:PWR_FLAG #FLG02
 U 1 1 61953527
 P 3325 1300
-F 0 "#FLG0102" H 3325 1375 50  0001 C CNN
+F 0 "#FLG02" H 3325 1375 50  0001 C CNN
 F 1 "PWR_FLAG" H 3325 1473 50  0000 C CNN
 F 2 "" H 3325 1300 50  0001 C CNN
